Commit message: whole_body test 1

File: robots/hsrb4s.obj.urdf (robot description, URDF)
Before this commit: robot hsrb, 45 links, 44 joints
Links:
- added link odom_tmp, mass 0.10
- added link odom_xr_link, mass 0.10
- added link odom_yx_link, mass 0.10
Joints:
- added joint odom_r: type revolute, parent odom_xr_link, child odom_tmp, axis 0 0 1, limit lower=-3.1416 upper=3.1416 effort=0.1 velocity=1.0
- added joint odom_x: type prismatic, parent base_footprint, child odom_yx_link, axis 1 0 0, limit lower=-10 upper=10 effort=0.1 velocity=0.2
- added joint odom_y: type prismatic, parent odom_yx_link, child odom_xr_link, axis 0 1 0, limit lower=-10 upper=10 effort=0.1 velocity=0.2

Commit message: save configuration for base movement

File: robots/hsrb4s.obj.urdf (robot description, URDF)
Before this commit: robot hsrb, 48 links, 47 joints
Links:
- removed link odom_tmp
- added link hand_eef_link
- added link internal_odom, mass 0.10
Joints:
- added joint hand_eef_joint: type fixed, parent hand_palm_link, child hand_eef_link, origin xyz=0 0.0 0.0 rpy=0.0 -1.57079 0.0
- joint odom_r: child odom_tmp -> base_footprint; limit lower=-3.1416 upper=3.1416 effort=0.1 velocity=1.0 -> lower=-6.2832 upper=6.2832 effort=0.1 velocity=0.5
- joint odom_x: child odom_yx_link -> odom_xr_link; parent base_footprint -> odom_yx_link
- joint odom_y: child odom_xr_link -> odom_yx_link; parent odom_yx_link -> internal_odom
